File: Hardware/KeyBoy.brd (EAGLE design)
At the start: 33 x 60 mm, 62 parts, among them U1 ESP32-S2-MINI-1-N4, U2 TLV75533PDBVRDBV5_TEX-L, U3 STM1061N25WX6FSOT-23_STM-L, U4 MCP73831T-2ACI/OTSOT-23-5_MC-L, U5 DMG3415U-7, U6 PAM8302AASCRPAM8302AASCR_DIO-L, X1 FH12-24S-0.5SH

Commit message: updating hardware files
Parts:
- removed C10: 01u, rcl:C0603
- removed C9: 0.1u, rcl:C0603
- removed R18: 30k, rcl:R0603
- removed VR1: 10k, SparkFun-Resistors:TRIMPOT-SMD-3MM-CLOSED
- C12: value 10u -> 4u7
- R17: value 30k -> 100k; device rcl:R0603 -> rcl:R0402
- U1: value ESP32-S2-MINI-1-N4 -> ESP32-S3-MINI-1-N8
- U6: value PAM8302AASCRPAM8302AASCR_DIO-L -> NAU8315YGQFN20_4X4_NUV-L; device PAM8302AASCR:PAM8302AASCR_DIO-L -> NAU8315YG:QFN20_4X4_NUV-L
- moved R17 23.4 mm to (7.26, 5.21), flipped to the top
- moved FB1 10.5 mm to (30.1, 7.16), turned to 270 degrees
- moved FB2 9.61 mm to (31.6, 7.16), turned to 90 degrees
- moved C11 8.67 mm to (30.0, 15.5), turned to 90 degrees
- moved C14 8.56 mm to (27.6, 3.68)
- moved C13 8.39 mm to (27.6, 6.30), turned to 0 degrees
- moved C12 2.87 mm to (32.0, 15.5), turned to 90 degrees
- moved U6 0.36 mm to (26.9, 12.1), turned to 90 degrees
Connections:
- removed net AUD_OUT: U1.10, VR1.1
- removed net N$12: R17.2, U6.4
- removed net N$13: R18.2, U6.3
- removed net N$15: C10.1, R18.1
- removed net N$16: C9.2, VR1.2
- new net I2S_BCLK: U1.9, U6.6
- new net I2S_DIN: U1.11, U6.9
- new net I2S_EN: U1.12, U6.3
- new net I2S_FCLK: U1.10, U6.8
- new net N$17: U6.13
- new net N$8: FB2.2, U6.16
- net AMP_IN: now also U6.11, U6.14, U6.2; no longer U6.1, U6.6
- net GND: now also R17.1, U6.12, U6.17, U6.18, U6.19, U6.21, U6.4; no longer C10.2, U6.7, VR1.3
- net N$14: now also U6.7; no longer C9.1, R17.1
- net N$5: now also U6.20; no longer C13.1, U6.8
- net N$6: now also R17.2, U$2.3; no longer C14.1, FB2.2, U6.5
- net VO+: now also C13.1
- net VO-: now also C14.1
Routing:
- net VO-: track 3.43 -> 17.5 mm
- net AMP_IN: track 35.9 -> 49.5 mm
- net GND: track 15.1 -> 28.2 mm, vias 17 -> 18
- net I2S_EN: track 0.00 -> 10.9 mm, vias 0 -> 1
- net VO+: track 10.6 -> 20.6 mm
- net AUD_OUT: track 8.75 -> 0.00 mm, vias 1 -> 0
- net N$8: track 0.00 -> 7.66 mm
- net I2S_FCLK: track 0.00 -> 7.50 mm, vias 0 -> 1
- net I2S_BCLK: track 0.00 -> 6.86 mm, vias 0 -> 1
- net I2S_DIN: track 0.00 -> 4.89 mm, vias 0 -> 1
- net N$13: track 4.06 -> 0.00 mm
- net RESET: track 25.7 -> 29.6 mm
- net N$6: track 4.32 -> 1.51 mm
- net N$16: track 2.24 -> 0.00 mm
- net N$14: track 1.77 -> 0.00 mm
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