File: Hardware/KeyBoy.sch (EAGLE design)
At the start: 62 parts, among them U1 ESP32-S2-MINI-1-N4, U2 TLV75533PDBVRDBV5_TEX-L, U3 STM1061N25WX6FSOT-23_STM-L, U4 MCP73831T-2ACI/OTSOT-23-5_MC-L, U5 DMG3415U-7, U6 PAM8302AASCRPAM8302AASCR_DIO-L, X1 FH12-24S-0.5SH

Commit message: updating hardware files
Parts:
- removed C10: 01u, rcl:C-USC0603
- removed C9: 0.1u, rcl:C-USC0603
- removed R18: 30k, rcl:R-US_R0603
- removed VR1: 10k, SparkFun-Resistors:TRIMPOT-SMD-3MM-CLOSED-1/8W-20%
- C12: value 10u -> 4u7
- R17: value 30k -> 100k; device rcl:R-US_R0603 -> rcl:R-US_R0402
- U1: value ESP32-S2-MINI-1-N4 -> ESP32-S3-MINI-1-N8
- U6: value PAM8302AASCRPAM8302AASCR_DIO-L -> NAU8315YGQFN20_4X4_NUV-L; device PAM8302AASCR:PAM8302AASCRPAM8302AASCR_DIO-L -> NAU8315YG:NAU8315YGQFN20_4X4_NUV-L
Connections:
- removed net AUD_OUT: U1A.IO6, VR1.CCW
- removed net N$12: R17.2, U6.IN-
- removed net N$13: R18.2, U6.IN+
- removed net N$15: C10.1, R18.1
- removed net N$16: C9.2, VR1.WIPER
- new net I2S_BCLK: U1A.IO5, U6.BCLK
- new net I2S_DIN: U1A.IO7, U6.DACIN
- new net I2S_EN: U1A.IO8, U6.EN
- new net I2S_FCLK: U1A.IO6, U6.FSL
- new net N$17: U6.GAIN
- new net N$8: FB2.2, U6.OUTN
- net AMP_IN: now also U6.VDD_2, U6.VDD_3; no longer U6.!SD
- net GND: now also R17.1, U6.VSS, U6.VSS_2, U6.VSS_3, U6.VSS_4, U6.VSS_5, U6.VSS_6; no longer C10.2, U6.GND, VR1.CW
- net N$14: now also U6.FSR; no longer C9.1, R17.1
- net N$5: now also U6.OUTP; no longer C13.1, U6.VO-
- net N$6: now also R17.2, U$2.3; no longer C14.1, FB2.2, U6.VO+
- net VO+: now also C13.1
- net VO-: now also C14.1
Other:
- moved on the sheet: C13, C14
